File: Circuit Design/Schematic/Schematic.sch (KiCad schematic (older format))
At the start: 3 parts, among them U1 ESP8266-12E_ESP-12E

Commit message: ESP changed
Parts:
- removed U1: ESP8266-12E_ESP-12E, XCVR_ESP8266-12E/ESP-12E, symbol ESP8266-12E_ESP-12E:ESP8266-12E_ESP-12E
- added U1: ESP32-WROOM-32, RF_Module:ESP32-WROOM-32, symbol RF_Module:ESP32-WROOM-32
Changed lines of the file:
@@
 Comment4 ""
 $EndDescr
-$Comp
-L ESP8266-12E_ESP-12E:ESP8266-12E_ESP-12E U1
-U 1 1 6259BF87
-P 6350 3550
-F 0 "U1" H 6350 4417 50  0000 C CNN
-F 1 "ESP8266-12E_ESP-12E" H 6350 4326 50  0000 C CNN
-F 2 "XCVR_ESP8266-12E/ESP-12E" H 6350 3550 50  0001 L BNN
-F 3 "" H 6350 3550 50  0001 L BNN
-F 4 "AI-Thinker" H 6350 3550 50  0001 L BNN "MANUFACTURER"
-	1    6350 3550
-	1    0    0    -1
-$EndComp
-Text HLabel 7175 2950 2    50   Input ~ 0
-3v3
-Wire Wire Line
-	7175 2950 7050 2950
 $Sheet
 S 2225 1225 775  775
@@
 F6 "R_Gnd" I L 2225 1825 50
 $EndSheet
-$Comp
-L power:GND #PWR?
-U 1 1 625A0879
-P 7150 4250
-F 0 "#PWR?" H 7150 4000 50  0001 C CNN
-F 1 "GND" H 7155 4077 50  0000 C CNN
-F 2 "" H 7150 4250 50  0001 C CNN
-F 3 "" H 7150 4250 50  0001 C CNN
-	1    7150 4250
-	1    0    0    -1
-$EndComp
-Wire Wire Line
-	7150 4250 7050 4250
 $Comp
 L Connector:Conn_01x03_Male Conn_Power
@@
 Wire Wire Line
 	2175 3300 1950 3300
-Text GLabel 7175 3250 2    50   Output ~ 0
+$Comp
+L RF_Module:ESP32-WROOM-32 U1
+U 1 1 626B0839
+P 5675 3150
+F 0 "U1" H 5675 4731 50  0000 C CNN
+F 1 "ESP32-WROOM-32" H 5675 4640 50  0000 C CNN
+F 2 "RF_Module:ESP32-WROOM-32" H 5675 1650 50  0001 C CNN
+F 3 "https://www.espressif.com/sites/default/files/documentation/esp32-wroom-32_datasheet_en.pdf" H 5375 3200 50  0001 C CNN
+	1    5675 3150
+	1    0    0    -1
+$EndComp
+Text GLabel 6400 2250 2    50   Input ~ 0
+Prog_Tx
+Wire Wire Line
+	6400 2250 6275 2250
+Text GLabel 6400 2050 2    50   Output ~ 0
 Prog_Rx
 Wire Wire Line
-	7050 3250 7175 3250
-Text GLabel 5475 3150 0    50   Input ~ 0
-Prog_Tx
+	6400 2050 6275 2050
+Text HLabel 5800 1750 2    50   Input ~ 0
+3v3
 Wire Wire Line
-	5475 3150 5650 3150
+	5675 1750 5800 1750
+$Comp
+L power:GND #PWR?
+U 1 1 626B993A
+P 5675 4625
+F 0 "#PWR?" H 5675 4375 50  0001 C CNN
+F 1 "GND" H 5680 4452 50  0000 C CNN
+F 2 "" H 5675 4625 50  0001 C CNN
+F 3 "" H 5675 4625 50  0001 C CNN
+	1    5675 4625
+	1    0    0    -1
+$EndComp
+Wire Wire Line
+	5675 4625 5675 4550
 $EndSCHEMATC

Commit message: minor changes
Parts:
- added R?: R, symbol Device:R
- added SW?: SW_DIP_x01, symbol Switch:SW_DIP_x01
Connections:
- net 3v3: now also R?.1
- net GND: now also SW?.1
- net at U1.3 (EN): now also R?.2, SW?.2
Changed lines of the file:
@@
 Wire Wire Line
 	5675 4625 5675 4550
+$Comp
+L Switch:SW_DIP_x01 SW?
+U 1 1 626C84CB
+P 4650 1950
+F 0 "SW?" H 4650 2217 50  0000 C CNN
+F 1 "SW_DIP_x01" H 4650 2126 50  0000 C CNN
+F 2 "" H 4650 1950 50  0001 C CNN
+F 3 "~" H 4650 1950 50  0001 C CNN
+	1    4650 1950
+	1    0    0    -1
+$EndComp
+$Comp
+L power:GND #PWR?
+U 1 1 626CCBB2
+P 4350 2050
+F 0 "#PWR?" H 4350 1800 50  0001 C CNN
+F 1 "GND" H 4355 1877 50  0000 C CNN
+F 2 "" H 4350 2050 50  0001 C CNN
+F 3 "" H 4350 2050 50  0001 C CNN
+	1    4350 2050
+	1    0    0    -1
+$EndComp
+Wire Wire Line
+	4350 1950 4350 2050
+Wire Wire Line
+	4950 1950 5025 1950
+Text HLabel 5025 1500 2    50   Input ~ 0
+3v3
+$Comp
+L Device:R R?
+U 1 1 626D4D5A
+P 5025 1750
+F 0 "R?" H 5095 1796 50  0000 L CNN
+F 1 "R" H 5095 1705 50  0000 L CNN
+F 2 "" V 4955 1750 50  0001 C CNN
+F 3 "~" H 5025 1750 50  0001 C CNN
+	1    5025 1750
+	1    0    0    -1
+$EndComp
+Wire Wire Line
+	5025 1500 5025 1600
+Wire Wire Line
+	5025 1900 5025 1950
+Connection ~ 5025 1950
+Wire Wire Line
+	5025 1950 5075 1950
 $EndSCHEMATC

Commit message: Minor changes
Parts:
- added ESP_Prog_Enable: SW_DIP_x01, symbol Switch:SW_DIP_x01
- added LED_prog: LED, symbol Device:LED
- added R_prog: R, symbol Device:R
- gave numbers to parts that had none: 1
Connections:
- net GND: now also ESP_Prog_Enable.2, LED_prog.1 (K)
- net at U1.16 (IO13): now also R_prog.2
- net at U1.25 (IO0): now also ESP_Prog_Enable.1
- new net: LED_prog.2 (A), R_prog.1
Changed lines of the file:
@@
 	5675 4625 5675 4550
 $Comp
-L Switch:SW_DIP_x01 SW?
+L Switch:SW_DIP_x01 ESP_Reset
 U 1 1 626C84CB
 P 4650 1950
-F 0 "SW?" H 4650 2217 50  0000 C CNN
+F 0 "ESP_Reset" H 4650 2217 50  0000 C CNN
 F 1 "SW_DIP_x01" H 4650 2126 50  0000 C CNN
 F 2 "" H 4650 1950 50  0001 C CNN
@@
 Wire Wire Line
 	5025 1950 5075 1950
+$Comp
+L Switch:SW_DIP_x01 ESP_Prog_Enable
+U 1 1 626D6A20
+P 6625 1825
+F 0 "ESP_Prog_Enable" H 6625 2092 50  0000 C CNN
+F 1 "SW_DIP_x01" H 6625 2001 50  0000 C CNN
+F 2 "" H 6625 1825 50  0001 C CNN
+F 3 "~" H 6625 1825 50  0001 C CNN
+	1    6625 1825
+	1    0    0    -1
+$EndComp
+Wire Wire Line
+	6325 1825 6300 1825
+Wire Wire Line
+	6300 1825 6300 1950
+Wire Wire Line
+	6300 1950 6275 1950
+$Comp
+L power:GND #PWR?
+U 1 1 626D7EE3
+P 7000 1825
+F 0 "#PWR?" H 7000 1575 50  0001 C CNN
+F 1 "GND" H 7005 1652 50  0000 C CNN
+F 2 "" H 7000 1825 50  0001 C CNN
+F 3 "" H 7000 1825 50  0001 C CNN
+	1    7000 1825
+	1    0    0    -1
+$EndComp
+Wire Wire Line
+	6925 1825 7000 1825
+$Comp
+L Device:LED LED_prog
+U 1 1 626D97DE
+P 6775 2650
+F 0 "LED_prog" H 6550 2650 50  0000 C CNN
+F 1 "LED" H 6400 2600 50  0001 C CNN
+F 2 "" H 6775 2650 50  0001 C CNN
+F 3 "~" H 6775 2650 50  0001 C CNN
+	1    6775 2650
+	-1   0    0    1
+$EndComp
+$Comp
+L power:GND #PWR?
+U 1 1 626DDABC
+P 7250 2650
+F 0 "#PWR?" H 7250 2400 50  0001 C CNN
+F 1 "GND" V 7255 2522 50  0000 R CNN
+F 2 "" H 7250 2650 50  0001 C CNN
+F 3 "" H 7250 2650 50  0001 C CNN
+	1    7250 2650
+	0    -1   -1   0
+$EndComp
+$Comp
+L Device:R R_prog
+U 1 1 626E07EA
+P 6475 2650
+F 0 "R_prog" V 6475 2675 50  0000 C CNN
+F 1 "R" V 6359 2650 50  0001 C CNN
+F 2 "" V 6405 2650 50  0001 C CNN
+F 3 "~" H 6475 2650 50  0001 C CNN
+	1    6475 2650
+	0    1    1    0
+$EndComp
+Wire Wire Line
+	6325 2650 6275 2650
+Wire Wire Line
+	6925 2650 7250 2650
 $EndSCHEMATC

Commit message: minor changes
Parts:
- R_prog: value R -> 39
- R_up_en: renamed from R?; value R -> 10k
Changed lines of the file:
@@
 U 1 1 626B0839
 P 5675 3150
-F 0 "U1" H 5675 4731 50  0000 C CNN
-F 1 "ESP32-WROOM-32" H 5675 4640 50  0000 C CNN
+F 0 "U1" H 5475 3675 50  0000 C CNN
+F 1 "ESP32-WROOM-32" H 5575 3500 50  0000 C CNN
 F 2 "RF_Module:ESP32-WROOM-32" H 5675 1650 50  0001 C CNN
 F 3 "https://www.espressif.com/sites/default/files/documentation/esp32-wroom-32_datasheet_en.pdf" H 5375 3200 50  0001 C CNN
@@
 Text HLabel 5025 1500 2    50   Input ~ 0
 3v3
-$Comp
-L Device:R R?
-U 1 1 626D4D5A
-P 5025 1750
-F 0 "R?" H 5095 1796 50  0000 L CNN
-F 1 "R" H 5095 1705 50  0000 L CNN
-F 2 "" V 4955 1750 50  0001 C CNN
-F 3 "~" H 5025 1750 50  0001 C CNN
-	1    5025 1750
-	1    0    0    -1
-$EndComp
 Wire Wire Line
 	5025 1500 5025 1600
@@
 P 6475 2650
 F 0 "R_prog" V 6475 2675 50  0000 C CNN
-F 1 "R" V 6359 2650 50  0001 C CNN
+F 1 "39" V 6359 2650 50  0001 C CNN
 F 2 "" V 6405 2650 50  0001 C CNN
 F 3 "~" H 6475 2650 50  0001 C CNN
@@
 Wire Wire Line
 	6925 2650 7250 2650
+$Comp
+L Device:R R_up_en
+U 1 1 626D4D5A
+P 5025 1750
+F 0 "R_up_en" H 5095 1750 50  0000 L CNN
+F 1 "10k" H 5095 1705 50  0001 L CNN
+F 2 "" V 4955 1750 50  0001 C CNN
+F 3 "~" H 5025 1750 50  0001 C CNN
+	1    5025 1750
+	1    0    0    -1
+$EndComp
 $EndSCHEMATC
