File: Circuit Design/Schematic/Schematic.sch (KiCad schematic (older format))
At the start: 8 parts, among them U1 ESP32-WROOM-32

Commit message: IDK
Parts:
- added J? (x2): Conn_01x03, symbol Connector_Generic:Conn_01x03
- added J_Lector_1, J_Lector_2, J_Lector_3: Conn_01x08, symbol Connector_Generic:Conn_01x08
Connections:
- wire segments 28 -> 41
Other:
- note added: "Los pines para los lectores están en este orden:\n1. SDA (SC)\n2. SCK\n3. MOSI\n4. MISO\n5. RQ\n6. GND\n7. RST\n8. 3V3\n"
