File: Circuit Design/Schematic/Schematic.kicad_sch (KiCad schematic)
At the start: 13 parts, among them U1 ESP32-WROOM-32

Commit message: Motor Schematic
Se incluye el esquemático del motor junto con algunas funciones, como condensador de bypass y elementos de antirrebote
Parts:
- removed R_up_en: 10k, symbol Device:R
- added C1, C3, C_Bypass: 100n, symbol pspice:CAP
- added R2, R3, R4: 10K, symbol Device:R
Connections:
- net 3v3: now also C_Bypass.2, R2.1, R3.2
- net GND: now also J_Motor_1.3 (Pin_3), J_Motor_2.3 (Pin_3), C1.2, C3.1, C_Bypass.1
- net at U1.25 (IO0): now also C3.2, R3.1, R4.2; no longer ESP_Prog_Enable.1
- net PWM_M1: now reaches U1.27 (IO16)
- net PWM_M1: now also J_Motor_1.1 (Pin_1)
- net PWM_M2: now reaches U1.28 (IO17)
- net PWM_M2: now also J_Motor_2.1 (Pin_1)
- net at ESP_Reset.2, U1.3 (EN): now also C1.1, R2.2
- net 5v0: now reaches J_Motor_2.2 (Pin_2)
- net 5v0: now also J_Motor_1.2 (Pin_2)
- new net: ESP_Prog_Enable.1, R4.1
Other:
- moved on the sheet: ESP_Prog_Enable, ESP_Reset, J_Motor_1, J_Motor_2
