File: Circuit Design/Schematic Test/TestEasyrun/TestEasyrun.kicad_sch (KiCad schematic)
At the start: 28 parts, among them U1 ESP32-WROOM-32

Commit message: Botón de rst
Se arreglaron las resistencias del botón de reset y enable
Parts:
- added C5, C6: 100n, Capacitor_SMD:C_0805_2012Metric_Pad1.18x1.45mm_HandSolder, symbol pspice:CAP
- added R6: 220, Resistor_SMD:R_0805_2012Metric_Pad1.20x1.40mm_HandSolder, symbol Device:R
- added R7, R8: 10K, Resistor_SMD:R_0805_2012Metric_Pad1.20x1.40mm_HandSolder, symbol Device:R
- R5: value 10K -> 220
Connections:
- net 3v3: now also C5.2, C6.2, R7.1, R8.1
- net Butt_D: now also C6.1
- net Butt_No_D: now also C5.1
- net I2C1: now also R8.2
- net I2C2: now also R7.2
- net at C1.1, R1.2, U1.3 (EN): now also R6.1; no longer ESP_Reset1.2
- new net: ESP_Reset1.2, R6.2
Other:
- moved on the sheet: C1, ESP_Reset1, J_Tap_1, J_Tap_2, J_gnd
