File: Circuit Design/Schematic Test/TestEasyrun/PWM_Generator_3v3.kicad_sch (KiCad schematic)
At the start: 12 parts

Commit message: Change the global labels
Connections:
- net Vo_rec is gone; now on net Vrec: DBT_3v3.2 (A)
- net Vs_3v3: now reaches CBT_3v3.2, Driver_3v3.4 (HS)
Changed lines of the file:
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@@
   (junction (at 127.635 100.33) (diameter 0) (color 0 0 0 0)
+  )
+  (junction (at 180.975 104.775) (diameter 0) (color 0 0 0 0)
   )
   (no_connect (at 90.17 93.98))
@@
     (stroke (width 0) (type default) (color 0 0 0 0))
   )
+  (wire (pts (xy 180.975 104.775) (xy 180.975 106.68))
+    (stroke (width 0) (type default) (color 0 0 0 0))
+  )
   (wire (pts (xy 88.265 86.36) (xy 90.17 86.36))
     (stroke (width 0) (type default) (color 0 0 0 0))
@@
     (stroke (width 0) (type default) (color 0 0 0 0))
   )
-  (wire (pts (xy 183.515 104.775) (xy 179.07 104.775))
+  (wire (pts (xy 183.515 104.775) (xy 180.975 104.775))
     (stroke (width 0) (type default) (color 0 0 0 0))
   )
@@
   )
   (wire (pts (xy 127.635 91.44) (xy 130.81 91.44))
+    (stroke (width 0) (type default) (color 0 0 0 0))
+  )
+  (wire (pts (xy 180.975 104.775) (xy 179.07 104.775))
     (stroke (width 0) (type default) (color 0 0 0 0))
   )
@@
     (effects (font (size 1.27 1.27)) (justify right))
   )
+  (hierarchical_label "Vs_3v3" (shape input) (at 180.975 106.68 270)
+    (effects (font (size 1.27 1.27)) (justify right))
+  )
   (hierarchical_label "Vrec" (shape input) (at 222.25 80.645 0)
     (effects (font (size 1.27 1.27)) (justify left))
   )
-  (hierarchical_label "Vo_rec" (shape input) (at 169.545 104.775 270)
-    (effects (font (size 1.27 1.27)) (justify right))
-  )
+  (hierarchical_label "Vrec" (shape input) (at 169.545 104.775 270)
+    (effects (font (size 1.27 1.27)) (justify right))
+  )

Commit message: Labels
Connections:
- net Ref3v3_3v3 is gone; now on net Ref_3v3: Rdiv1_3v3.1, Rdiv2_3v3.2, U_PWM_3v3.15 (2IN−), U_PWM_3v3.2 (1IN−)
- net Ref_3v3: no longer Rdiv2_3v3.1, U_PWM_3v3.14 (REF)
- new net: Rdiv2_3v3.1, U_PWM_3v3.14 (REF)
Changed lines of the file:
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@@
   (junction (at 125.73 82.55) (diameter 0) (color 0 0 0 0)
   )
-  (junction (at 127.635 91.44) (diameter 0) (color 0 0 0 0)
-  )
   (junction (at 88.265 81.28) (diameter 0) (color 0 0 0 0)
   )
@@
   (junction (at 125.73 87.63) (diameter 0) (color 0 0 0 0)
   )
+  (junction (at 127.635 100.965) (diameter 0) (color 0 0 0 0)
+  )
   (junction (at 72.39 91.44) (diameter 0) (color 0 0 0 0)
   )
   (junction (at 128.27 79.375) (diameter 0) (color 0 0 0 0)
-  )
-  (junction (at 127.635 100.33) (diameter 0) (color 0 0 0 0)
   )
   (junction (at 180.975 104.775) (diameter 0) (color 0 0 0 0)
@@
     (stroke (width 0) (type default) (color 0 0 0 0))
   )
-  (wire (pts (xy 127.635 100.33) (xy 127.635 99.695))
+  (wire (pts (xy 127.635 99.695) (xy 127.635 100.965))
     (stroke (width 0) (type default) (color 0 0 0 0))
   )
@@
     (stroke (width 0) (type default) (color 0 0 0 0))
   )
-  (wire (pts (xy 127.635 100.33) (xy 127.635 101.6))
-    (stroke (width 0) (type default) (color 0 0 0 0))
-  )
-  (wire (pts (xy 127.635 91.44) (xy 130.81 91.44))
-    (stroke (width 0) (type default) (color 0 0 0 0))
-  )
   (wire (pts (xy 180.975 104.775) (xy 179.07 104.775))
     (stroke (width 0) (type default) (color 0 0 0 0))
@@
     (stroke (width 0) (type default) (color 0 0 0 0))
   )
-  (wire (pts (xy 127.635 100.33) (xy 130.81 100.33))
-    (stroke (width 0) (type default) (color 0 0 0 0))
-  )
   (wire (pts (xy 86.995 83.82) (xy 86.995 86.36))
     (stroke (width 0) (type default) (color 0 0 0 0))
@@
     (stroke (width 0) (type default) (color 0 0 0 0))
   )
+  (wire (pts (xy 127.635 100.965) (xy 130.175 100.965))
+    (stroke (width 0) (type default) (color 0 0 0 0))
+  )
   (wire (pts (xy 88.265 81.28) (xy 90.17 81.28))
     (stroke (width 0) (type default) (color 0 0 0 0))
@@
     (stroke (width 0) (type default) (color 0 0 0 0))
   )
+  (wire (pts (xy 127.635 100.965) (xy 127.635 101.6))
+    (stroke (width 0) (type default) (color 0 0 0 0))
+  )
   (wire (pts (xy 90.17 106.68) (xy 87.63 106.68))
     (stroke (width 0) (type default) (color 0 0 0 0))
@@
     (stroke (width 0) (type default) (color 0 0 0 0))
   )
-  (global_label "Ref3v3_3v3" (shape input) (at 130.81 100.33 0) (fields_autoplaced)
-    (effects (font (size 1.27 1.27)) (justify left))
-    (property "Intersheet References" "${INTERSHEET_REFS}" (id 0) (at 144.0483 100.2506 0)
-      (effects (font (size 1.27 1.27)) (justify left) hide)
-    )
-  )
-  (global_label "Ref3v3_3v3" (shape input) (at 85.09 86.36 180) (fields_autoplaced)
-    (effects (font (size 1.27 1.27)) (justify right))
-    (property "Intersheet References" "${INTERSHEET_REFS}" (id 0) (at 71.8517 86.2806 0)
-      (effects (font (size 1.27 1.27)) (justify right) hide)
-    )
-  )
-  (global_label "Ref_3v3" (shape output) (at 130.81 91.44 0) (fields_autoplaced)
-    (effects (font (size 1.27 1.27)) (justify left))
-    (property "Intersheet References" "${INTERSHEET_REFS}" (id 0) (at 140.6617 91.3606 0)
-      (effects (font (size 1.27 1.27)) (justify left) hide)
-    )
+  (label "PWM_3v3" (at 127.635 87.63 0)
+    (effects (font (size 1.27 1.27)) (justify left bottom))
+  )
+  (label "Ref_3v3" (at 85.09 86.36 180)
+    (effects (font (size 1.27 1.27)) (justify right bottom))
+  )
+  (label "PWM_3v3" (at 182.245 85.725 180)
+    (effects (font (size 1.27 1.27)) (justify right bottom))
+  )
+  (label "Ref_3v3" (at 130.175 100.965 0)
+    (effects (font (size 1.27 1.27)) (justify left bottom))
   )
   (global_label "Ref_3v3" (shape input) (at 56.515 103.505 270) (fields_autoplaced)
@@
       (effects (font (size 1.27 1.27)) (justify right) hide)
     )
-  )
-  (global_label "PWM_3v3" (shape output) (at 127.635 87.63 0) (fields_autoplaced)
-    (effects (font (size 1.27 1.27)) (justify left))
-    (property "Intersheet References" "${INTERSHEET_REFS}" (id 0) (at 138.5752 87.5506 0)
-      (effects (font (size 1.27 1.27)) (justify left) hide)
-    )
-  )
-  (global_label "PWM_3v3" (shape input) (at 182.245 85.725 180) (fields_autoplaced)
-    (effects (font (size 1.27 1.27)) (justify right))
-    (property "Intersheet References" "${INTERSHEET_REFS}" (id 0) (at 171.3048 85.6456 0)
-      (effects (font (size 1.27 1.27)) (justify right) hide)
-    )
