File: Circuit Design/Schematic Test/TestEasyrun/PWM_Generator_5v0.kicad_sch (KiCad schematic)
At the start: 10 parts

Commit message: Change the global labels
Connections:
- net Vs_5v0: now reaches CBT_5v0.2, Driver_5v0.4 (HS)
Changed lines of the file:
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@@
 (kicad_sch (version 20211123) (generator eeschema)
   (paper "A4")
+  (junction (at 182.245 104.14) (diameter 0) (color 0 0 0 0)
+  )
   (junction (at 135.89 78.74) (diameter 0) (color 0 0 0 0)
   )
@@
     (stroke (width 0) (type default) (color 0 0 0 0))
   )
-  (wire (pts (xy 184.785 104.14) (xy 179.07 104.14))
+  (wire (pts (xy 184.785 104.14) (xy 182.245 104.14))
     (stroke (width 0) (type default) (color 0 0 0 0))
   )
@@
     (stroke (width 0) (type default) (color 0 0 0 0))
   )
+  (wire (pts (xy 182.245 104.14) (xy 182.245 106.045))
+    (stroke (width 0) (type default) (color 0 0 0 0))
+  )
   (wire (pts (xy 80.01 90.805) (xy 80.01 92.075))
     (stroke (width 0) (type default) (color 0 0 0 0))
@@
   )
   (wire (pts (xy 165.1 86.36) (xy 165.1 88.265))
+    (stroke (width 0) (type default) (color 0 0 0 0))
+  )
+  (wire (pts (xy 182.245 104.14) (xy 179.07 104.14))
     (stroke (width 0) (type default) (color 0 0 0 0))
   )
@@
     (effects (font (size 1.27 1.27)) (justify left))
   )
+  (hierarchical_label "Vs_5v0" (shape input) (at 182.245 106.045 270)
+    (effects (font (size 1.27 1.27)) (justify right))
+  )
   (hierarchical_label "Vrec" (shape input) (at 170.18 102.87 270)

Commit message: Labels
Connections:
- net Vo_rec is gone; now on net Vrec: Driver_5v0.1 (VDD)
Changed lines of the file:
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@@
     (stroke (width 0) (type default) (color 0 0 0 0))
   )
-  (global_label "Ref_5v0" (shape output) (at 135.255 90.805 0) (fields_autoplaced)
-    (effects (font (size 1.27 1.27)) (justify left))
-    (property "Intersheet References" "${INTERSHEET_REFS}" (id 0) (at 145.1067 90.7256 0)
-      (effects (font (size 1.27 1.27)) (justify left) hide)
-    )
+  (label "Ref_5v0" (at 135.255 90.805 0)
+    (effects (font (size 1.27 1.27)) (justify left bottom))
   )
-  (global_label "Ref_5v0" (shape input) (at 92.71 85.725 180) (fields_autoplaced)
-    (effects (font (size 1.27 1.27)) (justify right))
-    (property "Intersheet References" "${INTERSHEET_REFS}" (id 0) (at 82.8583 85.6456 0)
-      (effects (font (size 1.27 1.27)) (justify right) hide)
-    )
+  (label "Ref_5v0" (at 64.77 102.87 270)
+    (effects (font (size 1.27 1.27)) (justify right bottom))
   )
-  (global_label "PWM_5v0" (shape output) (at 135.255 86.995 0) (fields_autoplaced)
-    (effects (font (size 1.27 1.27)) (justify left))
-    (property "Intersheet References" "${INTERSHEET_REFS}" (id 0) (at 146.1952 86.9156 0)
-      (effects (font (size 1.27 1.27)) (justify left) hide)
-    )
+  (label "Ref_5v0" (at 92.71 85.725 180)
+    (effects (font (size 1.27 1.27)) (justify right bottom))
   )
-  (global_label "Ref_5v0" (shape input) (at 64.77 102.87 270) (fields_autoplaced)
-    (effects (font (size 1.27 1.27)) (justify right))
-    (property "Intersheet References" "${INTERSHEET_REFS}" (id 0) (at 64.6906 112.7217 90)
-      (effects (font (size 1.27 1.27)) (justify right) hide)
-    )
+  (label "PWM_5v0" (at 135.255 86.995 0)
+    (effects (font (size 1.27 1.27)) (justify left bottom))
   )
-  (global_label "PWM_5v0" (shape input) (at 185.42 83.82 180) (fields_autoplaced)
-    (effects (font (size 1.27 1.27)) (justify right))
-    (property "Intersheet References" "${INTERSHEET_REFS}" (id 0) (at 174.4798 83.7406 0)
-      (effects (font (size 1.27 1.27)) (justify right) hide)
-    )
-  )
-  (global_label "Vo_rec" (shape input) (at 221.615 78.74 0) (fields_autoplaced)
-    (effects (font (size 1.27 1.27)) (justify left))
-    (property "Intersheet References" "${INTERSHEET_REFS}" (id 0) (at 230.1967 78.6606 0)
-      (effects (font (size 1.27 1.27)) (justify left) hide)
-    )
+  (label "PWM_5v0" (at 185.42 83.82 180)
+    (effects (font (size 1.27 1.27)) (justify right bottom))
   )
   (hierarchical_label "5v0_Ref" (shape input) (at 92.71 80.645 180)
     (effects (font (size 1.27 1.27)) (justify right))
   )
+  (hierarchical_label "Vrec" (shape input) (at 221.615 78.74 0)
+    (effects (font (size 1.27 1.27)) (justify left))
+  )
   (hierarchical_label "Vrec" (shape input) (at 137.16 78.74 0)
