File: Circuit Design/Schematic Test/TestEasyrun/PowerModule.kicad_sch (KiCad schematic)
At the start: 11 parts

Commit message: Labels
Other:
- moved on the sheet: C_Buck3v3, D_Buck3v3, L_Buck3v3, Q_3v3
