File: Circuit Design/Final Schematic/Easyrun.kicad_sch (KiCad schematic)
At the start: 20 parts, among them U1 ESP32-WROOM-32

Commit message: Footprints
Parts:
- J_I2C1: footprint Connector_PinHeader_2.54mm:PinHeader_1x05_P2.54mm_Vertical -> Connector_PinSocket_2.54mm:PinSocket_1x05_P2.54mm_Horizontal
- J_prog1: renamed from J_prog; footprint Connector_PinSocket_2.54mm:PinSocket_1x06_P2.54mm_Vertical -> Connector_PinHeader_2.54mm:PinHeader_1x06_P2.54mm_Horizontal
- renumbered BProg to BProg1, BRst to BRst1, CB to CB1, J_gnd to J_gnd1, LProg to LProg1, RMISO to RMISO1, R_prog to R_prog1

Commit message: PCB distribution
Parts:
- renumbered LProg1 to L_p1, R_prog1 to R_p1
Changed lines of the file:
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@@
   (symbol (lib_id "Device:LED") (at 92.71 88.9 90) (unit 1)
     (in_bom yes) (on_board yes)
-    (property "Reference" "LProg1" (id 0) (at 90.17 92.71 0))
+    (property "Reference" "L_p1" (id 0) (at 90.17 92.71 0))
     (property "Value" "LED" (id 1) (at 93.98 98.425 0)
       (effects (font (size 1.27 1.27)) hide)
@@
   (symbol (lib_id "Device:R") (at 92.71 81.28 180) (unit 1)
     (in_bom yes) (on_board yes)
-    (property "Reference" "R_prog1" (id 0) (at 90.17 83.82 90))
+    (property "Reference" "R_p1" (id 0) (at 90.17 83.82 90))
     (property "Value" "47" (id 1) (at 95.6564 81.28 90))
     (property "Footprint" "Resistor_SMD:R_0805_2012Metric_Pad1.20x1.40mm_HandSolder" (id 2) (at 94.488 81.28 90)
@@
       (reference "CByBa1") (unit 1) (value "10u") (footprint "Capacitor_SMD:CP_Elec_6.3x5.8")
     )
+    (path "/ce33739c-5d28-4c4f-8ccf-84b467a2a283/a95a8dfc-9f79-410d-a225-f43375e2a94b/9c674106-6c66-4027-bc63-5e55a554fc6b"
+      (reference "C_b1") (unit 1) (value "C_Polarized") (footprint "Capacitor_SMD:CP_Elec_6.3x5.8")
+    )
     (path "/ce33739c-5d28-4c4f-8ccf-84b467a2a283/a95a8dfc-9f79-410d-a225-f43375e2a94b/9000c85f-cb97-497a-b20c-46cf02358932"
       (reference "C_by1") (unit 1) (value "10n") (footprint "Capacitor_SMD:C_0805_2012Metric_Pad1.18x1.45mm_HandSolder")
     )
-    (path "/ce33739c-5d28-4c4f-8ccf-84b467a2a283/a95a8dfc-9f79-410d-a225-f43375e2a94b/9c674106-6c66-4027-bc63-5e55a554fc6b"
-      (reference "C_by_2") (unit 1) (value "C_Polarized") (footprint "Capacitor_SMD:CP_Elec_6.3x5.8")
-    )
     (path "/ce33739c-5d28-4c4f-8ccf-84b467a2a283/a95a8dfc-9f79-410d-a225-f43375e2a94b/9f43f97d-5da0-4635-9c3c-4c4ecc5e776b"
       (reference "C_cv1") (unit 1) (value "10n") (footprint "Capacitor_SMD:C_0805_2012Metric_Pad1.18x1.45mm_HandSolder")
@@
     )
     (path "/ce33739c-5d28-4c4f-8ccf-84b467a2a283/2742c4ea-a381-46e6-9108-7abf967d887e"
-      (reference "D1") (unit 1) (value "1N5822") (footprint "Diode_THT:D_DO-201AD_P15.24mm_Horizontal")
+      (reference "D1") (unit 1) (value "1N5822") (footprint "Diode_THT:D_DO-201AE_P5.08mm_Vertical_AnodeUp")
     )
     (path "/ce33739c-5d28-4c4f-8ccf-84b467a2a283/f0e54572-ce21-4288-9f09-e30e644463d7"
-      (reference "D2") (unit 1) (value "1N5822") (footprint "Diode_THT:D_DO-201AD_P15.24mm_Horizontal")
+      (reference "D2") (unit 1) (value "1N5822") (footprint "Diode_THT:D_DO-201AE_P5.08mm_Vertical_AnodeUp")
     )
     (path "/ce33739c-5d28-4c4f-8ccf-84b467a2a283/eb3bf10c-415f-4231-8fef-acb0a60d93a5"
@@
     )
     (path "/ce33739c-5d28-4c4f-8ccf-84b467a2a283/72439c1f-bc73-458c-9ac0-42c96ebc04b0"
-      (reference "D4") (unit 1) (value "1N5822") (footprint "Diode_THT:D_DO-201AD_P15.24mm_Horizontal")
+      (reference "D4") (unit 1) (value "1N5822") (footprint "Diode_THT:D_DO-201AE_P5.08mm_Vertical_AnodeUp")
     )
     (path "/ce33739c-5d28-4c4f-8ccf-84b467a2a283/5adccc16-4c06-49da-909a-8a4d1a5b2995/d9751148-af1e-418c-88ff-4f06a0a21baf"
-      (reference "DB3") (unit 1) (value "1N5822") (footprint "Diode_THT:D_DO-201AD_P15.24mm_Horizontal")
+      (reference "DB3") (unit 1) (value "1N5822") (footprint "Diode_THT:D_DO-201AE_P5.08mm_Vertical_AnodeUp")
     )
     (path "/ce33739c-5d28-4c4f-8ccf-84b467a2a283/47c3fd19-e8b0-4d87-ba69-8ede1ca5c801/d9751148-af1e-418c-88ff-4f06a0a21baf"
-      (reference "DB5") (unit 1) (value "1N5822") (footprint "Diode_THT:D_DO-201AD_P15.24mm_Horizontal")
+      (reference "DB5") (unit 1) (value "1N5822") (footprint "Diode_THT:D_DO-201AE_P5.08mm_Vertical_AnodeUp")
     )
     (path "/ce33739c-5d28-4c4f-8ccf-84b467a2a283/a95a8dfc-9f79-410d-a225-f43375e2a94b/30079145-2e0e-4c22-8e7c-788ec61e4444"
-      (reference "DBoo1") (unit 1) (value "1N5819") (footprint "Diode_THT:D_DO-41_SOD81_P10.16mm_Horizontal")
+      (reference "DBoo1") (unit 1) (value "1N5819") (footprint "Diode_THT:D_DO-201AE_P5.08mm_Vertical_AnodeUp")
     )
     (path "/ce33739c-5d28-4c4f-8ccf-84b467a2a283/118d15e0-06a7-423f-a72c-0cc161894136"
-      (reference "DFly1") (unit 1) (value "1N5822") (footprint "Diode_THT:D_DO-201AD_P15.24mm_Horizontal")
+      (reference "DFly1") (unit 1) (value "1N5822") (footprint "Diode_THT:D_DO-201AE_P5.08mm_Vertical_AnodeUp")
     )
     (path "/ce33739c-5d28-4c4f-8ccf-84b467a2a283/5ded5e05-91c3-4914-acd8-46f44022acc0/b4b31f94-7238-4ebb-8945-f8429e813474"
@@
     )
     (path "/ce33739c-5d28-4c4f-8ccf-84b467a2a283/ba09b7a2-59f0-45b6-95a4-046331578e0c"
-      (reference "D_S1") (unit 1) (value "1N5822") (footprint "Diode_THT:D_DO-201AD_P15.24mm_Horizontal")
+      (reference "D_S1") (unit 1) (value "1N5822") (footprint "Diode_THT:D_DO-201AE_P5.08mm_Vertical_AnodeUp")
     )
     (path "/ce33739c-5d28-4c4f-8ccf-84b467a2a283/105c7258-4162-4b7a-b521-952f194bc83b"
-      (reference "D_S2") (unit 1) (value "1N5822") (footprint "Diode_THT:D_DO-201AD_P15.24mm_Horizontal")
+      (reference "D_S2") (unit 1) (value "1N5822") (footprint "Diode_THT:D_DO-201AE_P5.08mm_Vertical_AnodeUp")
     )
     (path "/ce33739c-5d28-4c4f-8ccf-84b467a2a283/944023bb-0136-4552-b0c7-ccea65a609e4"
@@
     )
     (path "/250658cf-3442-4875-98b9-880ff77de779"
-      (reference "LProg1") (unit 1) (value "LED") (footprint "LED_SMD:LED_0805_2012Metric_Pad1.15x1.40mm_HandSolder")
+      (reference "L_p1") (unit 1) (value "LED") (footprint "LED_SMD:LED_0805_2012Metric_Pad1.15x1.40mm_HandSolder")
     )
     (path "/ce33739c-5d28-4c4f-8ccf-84b467a2a283/a95a8dfc-9f79-410d-a225-f43375e2a94b/86b9cc14-42fc-4a6c-8687-3339e1994761"
@@
     )
     (path "/6ee20d1c-a46d-41e5-9769-e0e93e111749"
-      (reference "R_prog1") (unit 1) (value "47") (footprint "Resistor_SMD:R_0805_2012Metric_Pad1.20x1.40mm_HandSolder")
+      (reference "R_p1") (unit 1) (value "47") (footprint "Resistor_SMD:R_0805_2012Metric_Pad1.20x1.40mm_HandSolder")
     )
     (path "/ce33739c-5d28-4c4f-8ccf-84b467a2a283/a95a8dfc-9f79-410d-a225-f43375e2a94b/ce62b4fd-c72d-403d-abc0-345bbc10d0b3"

Commit message: More free space schematic
Connections:
- net CS_Lector3: now also U1.24 (IO2); no longer U1.13 (IO14)
- net STDBY: now reaches U1.14 (IO12)
- new net CHRG: U1.13 (IO14)
- no-connect marks 13 -> 11
Changed lines of the file:
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@@
   (junction (at 150.495 86.36) (diameter 0) (color 0 0 0 0)
   )
-  (junction (at 180.975 55.88) (diameter 0) (color 0 0 0 0)
-  )
   (junction (at 45.72 120.65) (diameter 0) (color 0 0 0 0)
   )
@@
   )
   (junction (at 180.975 96.52) (diameter 0) (color 0 0 0 0)
-  )
-  (junction (at 180.975 71.12) (diameter 0) (color 0 0 0 0)
   )
   (junction (at 150.495 50.8) (diameter 0) (color 0 0 0 0)
@@
   (no_connect (at 148.59 88.9))
   (no_connect (at 148.59 83.82))
-  (no_connect (at 181.61 55.88))
   (no_connect (at 148.59 93.98))
-  (no_connect (at 182.245 66.04))
   (no_connect (at 148.59 58.42))
   (no_connect (at 55.245 86.36))
@@
     (stroke (width 0) (type default) (color 0 0 0 0))
   )
-  (wire (pts (xy 180.975 55.88) (xy 181.61 55.88))
-    (stroke (width 0) (type default) (color 0 0 0 0))
-  )
   (polyline (pts (xy 120.65 161.29) (xy 120.65 185.42))
     (stroke (width 0) (type default) (color 0 0 0 0))
@@
     (stroke (width 0) (type default) (color 0 0 0 0))
   )
+  (wire (pts (xy 180.975 55.88) (xy 184.15 55.88))
+    (stroke (width 0) (type default) (color 0 0 0 0))
+  )
   (wire (pts (xy 48.26 152.4) (xy 48.26 154.94))
     (stroke (width 0) (type default) (color 0 0 0 0))
@@
     (stroke (width 0) (type default) (color 0 0 0 0))
   )
-  (wire (pts (xy 180.975 66.04) (xy 182.245 66.04))
-    (stroke (width 0) (type default) (color 0 0 0 0))
-  )
   (wire (pts (xy 44.45 101.6) (xy 55.88 101.6))
     (stroke (width 0) (type default) (color 0 0 0 0))
@@
     (stroke (width 0) (type default) (color 0 0 0 0))
   )
-  (wire (pts (xy 180.34 55.88) (xy 180.975 55.88))
-    (stroke (width 0) (type default) (color 0 0 0 0))
-  )
   (wire (pts (xy 83.82 163.195) (xy 83.82 161.925))
     (stroke (width 0) (type default) (color 0 0 0 0))
@@
     (stroke (width 0) (type default) (color 0 0 0 0))
   )
+  (wire (pts (xy 180.975 66.04) (xy 190.5 66.04))
+    (stroke (width 0) (type default) (color 0 0 0 0))
+  )
   (wire (pts (xy 180.975 83.82) (xy 184.15 83.82))
     (stroke (width 0) (type default) (color 0 0 0 0))
@@
     (stroke (width 0) (type default) (color 0 0 0 0))
   )
+  (wire (pts (xy 180.975 71.12) (xy 194.31 71.12))
+    (stroke (width 0) (type default) (color 0 0 0 0))
+  )
   (polyline (pts (xy 82.55 107.95) (xy 82.55 66.04))
     (stroke (width 0) (type default) (color 0 0 0 0))
@@
     (stroke (width 0) (type default) (color 0 0 0 0))
   )
-  (wire (pts (xy 180.975 71.12) (xy 184.15 71.12))
-    (stroke (width 0) (type default) (color 0 0 0 0))
-  )
   (wire (pts (xy 212.09 120.65) (xy 224.79 120.65))
     (stroke (width 0) (type default) (color 0 0 0 0))
@@
   )
   (wire (pts (xy 44.45 104.14) (xy 55.88 104.14))
-    (stroke (width 0) (type default) (color 0 0 0 0))
-  )
-  (wire (pts (xy 180.34 71.12) (xy 180.975 71.12))
     (stroke (width 0) (type default) (color 0 0 0 0))
   )
@@
     (effects (font (size 1.27 1.27)) (justify left bottom))
   )
+  (label "CS_Lector3" (at 184.15 55.88 0)
+    (effects (font (size 1.27 1.27)) (justify left bottom))
+  )
   (label "Rst_D" (at 184.15 106.68 0)
     (effects (font (size 1.27 1.27)) (justify left bottom))
@@
     (effects (font (size 1.27 1.27)) (justify left bottom))
   )
-  (label "CS_Lector3" (at 184.15 71.12 0)
-    (effects (font (size 1.27 1.27)) (justify left bottom))
-  )
   (label "MISO" (at 212.09 53.34 0)
     (effects (font (size 1.27 1.27)) (justify left bottom))
@@
     (effects (font (size 1.27 1.27)) (justify right bottom))
   )
+  (global_label "CHRG" (shape input) (at 194.31 71.12 0) (fields_autoplaced)
+    (effects (font (size 1.27 1.27)) (justify left))
+    (property "Intersheet References" "${INTERSHEET_REFS}" (id 0) (at 201.8636 71.0406 0)
+      (effects (font (size 1.27 1.27)) (justify left) hide)
+    )
+  )
+  (global_label "STDBY" (shape input) (at 190.5 66.04 0) (fields_autoplaced)
+    (effects (font (size 1.27 1.27)) (justify left))
+    (property "Intersheet References" "${INTERSHEET_REFS}" (id 0) (at 198.7188 65.9606 0)
+      (effects (font (size 1.27 1.27)) (justify left) hide)
+    )
+  )
   (symbol (lib_id "power:GND") (at 56.515 83.82 90) (unit 1)
