File: Circuit Design/Final Schematic/Easyrun.kicad_sch (KiCad schematic)
At the start: 20 parts, among them U1 ESP32-WROOM-32

Commit message: Cambio orden pines lectores y display
Se cambiaron para facilitar el ruteo.
Connections:
- net CS_Display: now also U1.6 (IO34); no longer U1.23 (IO15)
- net CS_Lector2: now also U1.24 (IO2); no longer U1.36 (IO22)
- net CS_Lector3: now also U1.36 (IO22); no longer U1.24 (IO2)
- net D/C: now also U1.23 (IO15); no longer U1.7 (IO35)
- net Rst_D: now also U1.7 (IO35); no longer U1.6 (IO34)

Commit message: Corrección tamaño de vías
Se corrigió el tamaño de las vías pasantes de la PCB
Connections:
- net CS_Lector_1 is gone; now on net CS_Lector1: U1.29 (IO5)
Changed lines of the file:
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@@
     (effects (font (size 1.27 1.27)) (justify left bottom))
   )
-  (label "CS_Lector_1" (at 184.15 63.5 0)
+  (label "CS_Lector1" (at 184.15 63.5 0)
     (effects (font (size 1.27 1.27)) (justify left bottom))
   )

Commit message: Cambio pines CS y Rst Display
Se cambiaron los pines CS y Rst del Display que estaban en pines solo entrada de la ESP, por los pines STDBY y CHRG de la parte de potencia
Connections:
- net CHRG: now also U1.6 (IO34); no longer U1.13 (IO14)
- net CS_Display: now also U1.14 (IO12); no longer U1.6 (IO34)
- net Rst_D: now also U1.13 (IO14); no longer U1.7 (IO35)
- net STDBY: now also U1.7 (IO35); no longer U1.14 (IO12)
Changed lines of the file:
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@@
   (junction (at 180.975 76.2) (diameter 0) (color 0 0 0 0)
   )
+  (junction (at 180.975 71.12) (diameter 0) (color 0 0 0 0)
+  )
   (junction (at 48.26 152.4) (diameter 0) (color 0 0 0 0)
   )
@@
   (junction (at 150.495 58.42) (diameter 0) (color 0 0 0 0)
   )
+  (junction (at 180.975 109.22) (diameter 0) (color 0 0 0 0)
+  )
   (junction (at 45.72 109.22) (diameter 0) (color 0 0 0 0)
   )
@@
   (junction (at 150.495 86.36) (diameter 0) (color 0 0 0 0)
   )
+  (junction (at 180.975 106.68) (diameter 0) (color 0 0 0 0)
+  )
   (junction (at 45.72 120.65) (diameter 0) (color 0 0 0 0)
   )
@@
   )
   (junction (at 150.495 55.88) (diameter 0) (color 0 0 0 0)
+  )
+  (junction (at 180.975 66.04) (diameter 0) (color 0 0 0 0)
   )
   (junction (at 180.975 63.5) (diameter 0) (color 0 0 0 0)
@@
     (stroke (width 0) (type default) (color 0 0 0 0))
   )
+  (wire (pts (xy 180.34 106.68) (xy 180.975 106.68))
+    (stroke (width 0) (type default) (color 0 0 0 0))
+  )
   (wire (pts (xy 212.09 53.34) (xy 224.79 53.34))
     (stroke (width 0) (type default) (color 0 0 0 0))
@@
     (stroke (width 0) (type default) (color 0 0 0 0))
   )
+  (wire (pts (xy 180.34 71.12) (xy 180.975 71.12))
+    (stroke (width 0) (type default) (color 0 0 0 0))
+  )
   (wire (pts (xy 180.975 53.34) (xy 184.15 53.34))
     (stroke (width 0) (type default) (color 0 0 0 0))
@@
     (stroke (width 0) (type default) (color 0 0 0 0))
   )
+  (wire (pts (xy 180.34 66.04) (xy 180.975 66.04))
+    (stroke (width 0) (type default) (color 0 0 0 0))
+  )
   (wire (pts (xy 55.245 81.28) (xy 58.42 81.28))
     (stroke (width 0) (type default) (color 0 0 0 0))
@@
     (stroke (width 0) (type default) (color 0 0 0 0))
   )
+  (wire (pts (xy 180.975 71.12) (xy 184.15 71.12))
+    (stroke (width 0) (type default) (color 0 0 0 0))
+  )
   (wire (pts (xy 212.09 76.2) (xy 224.79 76.2))
     (stroke (width 0) (type default) (color 0 0 0 0))
@@
     (stroke (width 0) (type default) (color 0 0 0 0))
   )
-  (wire (pts (xy 183.515 106.68) (xy 180.975 106.68))
-    (stroke (width 0) (type default) (color 0 0 0 0))
-  )
   (wire (pts (xy 64.77 42.545) (xy 64.77 48.26))
     (stroke (width 0) (type default) (color 0 0 0 0))
@@
     (stroke (width 0) (type default) (color 0 0 0 0))
   )
+  (wire (pts (xy 180.34 109.22) (xy 180.975 109.22))
+    (stroke (width 0) (type default) (color 0 0 0 0))
+  )
   (wire (pts (xy 83.82 154.305) (xy 83.82 151.765))
     (stroke (width 0) (type default) (color 0 0 0 0))
@@
     (stroke (width 0) (type default) (color 0 0 0 0))
   )
+  (wire (pts (xy 180.975 106.68) (xy 184.15 106.68))
+    (stroke (width 0) (type default) (color 0 0 0 0))
+  )
   (polyline (pts (xy 111.76 57.15) (xy 41.91 57.15))
     (stroke (width 0) (type default) (color 0 0 0 0))
@@
     (stroke (width 0) (type default) (color 0 0 0 0))
   )
+  (wire (pts (xy 180.975 109.22) (xy 186.69 109.22))
+    (stroke (width 0) (type default) (color 0 0 0 0))
+  )
   (wire (pts (xy 55.245 83.82) (xy 56.515 83.82))
     (stroke (width 0) (type default) (color 0 0 0 0))
@@
     (stroke (width 0) (type default) (color 0 0 0 0))
   )
-  (wire (pts (xy 180.975 66.04) (xy 190.5 66.04))
-    (stroke (width 0) (type default) (color 0 0 0 0))
-  )
   (wire (pts (xy 180.975 83.82) (xy 184.15 83.82))
     (stroke (width 0) (type default) (color 0 0 0 0))
@@
     (stroke (width 0) (type default) (color 0 0 0 0))
   )
-  (wire (pts (xy 183.515 109.22) (xy 180.975 109.22))
-    (stroke (width 0) (type default) (color 0 0 0 0))
-  )
   (polyline (pts (xy 120.65 161.29) (xy 168.91 161.29))
     (stroke (width 0) (type default) (color 0 0 0 0))
   )
-  (wire (pts (xy 180.975 71.12) (xy 194.31 71.12))
-    (stroke (width 0) (type default) (color 0 0 0 0))
-  )
   (wire (pts (xy 180.975 73.66) (xy 184.15 73.66))
     (stroke (width 0) (type default) (color 0 0 0 0))
@@
   )
   (wire (pts (xy 148.59 88.9) (xy 150.495 88.9))
+    (stroke (width 0) (type default) (color 0 0 0 0))
+  )
+  (wire (pts (xy 180.975 66.04) (xy 184.15 66.04))
     (stroke (width 0) (type default) (color 0 0 0 0))
   )
@@
     (effects (font (size 1.27 1.27)) (justify left bottom))
   )
-  (label "Rst_D" (at 183.515 109.22 0)
-    (effects (font (size 1.27 1.27)) (justify left bottom))
-  )
   (label "Rst_3" (at 184.15 86.36 0)
     (effects (font (size 1.27 1.27)) (justify left bottom))
@@
   )
   (label "IO13" (at 184.15 68.58 0)
+    (effects (font (size 1.27 1.27)) (justify left bottom))
+  )
+  (label "Rst_D" (at 184.15 71.12 0)
     (effects (font (size 1.27 1.27)) (justify left bottom))
   )
@@
     (effects (font (size 1.27 1.27)) (justify left bottom))
   )
-  (label "CS_Display" (at 183.515 106.68 0)
-    (effects (font (size 1.27 1.27)) (justify left bottom))
-  )
   (label "CS_Lector1" (at 184.15 63.5 0)
     (effects (font (size 1.27 1.27)) (justify left bottom))
   )
   (label "Rst_3" (at 212.09 76.2 0)
+    (effects (font (size 1.27 1.27)) (justify left bottom))
+  )
+  (label "CS_Display" (at 184.15 66.04 0)
     (effects (font (size 1.27 1.27)) (justify left bottom))
   )
@@
     (effects (font (size 1.27 1.27)) (justify right bottom))
   )
-  (global_label "CHRG" (shape input) (at 194.31 71.12 0) (fields_autoplaced)
+  (global_label "CHRG" (shape input) (at 184.15 106.68 0) (fields_autoplaced)
     (effects (font (size 1.27 1.27)) (justify left))
-    (property "Intersheet References" "${INTERSHEET_REFS}" (id 0) (at 201.8636 71.0406 0)
+    (property "Intersheet References" "${INTERSHEET_REFS}" (id 0) (at 191.7036 106.6006 0)
       (effects (font (size 1.27 1.27)) (justify left) hide)
     )
   )
-  (global_label "STDBY" (shape input) (at 190.5 66.04 0) (fields_autoplaced)
+  (global_label "STDBY" (shape input) (at 186.69 109.22 0) (fields_autoplaced)
     (effects (font (size 1.27 1.27)) (justify left))
-    (property "Intersheet References" "${INTERSHEET_REFS}" (id 0) (at 198.7188 65.9606 0)
+    (property "Intersheet References" "${INTERSHEET_REFS}" (id 0) (at 194.9088 109.1406 0)
       (effects (font (size 1.27 1.27)) (justify left) hide)
     )
