File: Circuit Design/Final Schematic/Buck3v3.kicad_sch (KiCad schematic)
At the start: 5 parts

Commit message: Corrección tamaño de vías
Se corrigió el tamaño de las vías pasantes de la PCB
Parts:
- renumbered CB5 to CB3, CBy5 to CBy3, DB5 to DB3, LB5 to LB3, UB5v0 to UB3v3
Changed lines of the file:
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@@
   (symbol (lib_id "Device:C_Polarized") (at 126.365 93.98 0)
     (in_bom yes) (on_board yes)
-    (property "Reference" "CBy5" (id 0) (at 119.38 96.52 90)
+    (property "Reference" "CBy3" (id 0) (at 119.38 96.52 90)
       (effects (font (size 1.27 1.27)) (justify left))
     )
@@
   (symbol (lib_id "Device:C_Polarized") (at 189.865 101.6 0)
     (in_bom yes) (on_board yes) (fields_autoplaced)
-    (property "Reference" "CB5" (id 0) (at 193.04 99.4409 0)
+    (property "Reference" "CB3" (id 0) (at 193.04 99.4409 0)
       (effects (font (size 1.27 1.27)) (justify left))
     )
@@
   (symbol (lib_id "Device:L") (at 179.07 95.25 90)
     (in_bom yes) (on_board yes)
-    (property "Reference" "LB5" (id 0) (at 179.705 97.79 90))
+    (property "Reference" "LB3" (id 0) (at 179.705 97.79 90))
     (property "Value" "100u" (id 1) (at 179.705 100.33 90))
     (property "Footprint" "Inductor_THT:L_Toroid_Vertical_L25.4mm_W14.7mm_P12.20mm_Vishay_TJ5_BigPads" (id 2) (at 179.07 95.25 0)
@@
   (symbol (lib_id "Regulator_Switching:LM2576S-5") (at 146.05 92.71 0)
     (in_bom yes) (on_board yes) (fields_autoplaced)
-    (property "Reference" "UB5v0" (id 0) (at 146.05 82.55 0))
+    (property "Reference" "UB3v3" (id 0) (at 146.05 82.55 0))
     (property "Value" "LM2576S-5" (id 1) (at 146.05 85.09 0))
     (property "Footprint" "Package_TO_SOT_SMD:TO-263-5_TabPin3" (id 2) (at 146.05 99.06 0)
@@
   (symbol (lib_id "Diode:1N5822") (at 168.275 101.6 270)
     (in_bom yes) (on_board yes)
-    (property "Reference" "DB5" (id 0) (at 172.085 99.695 0)
+    (property "Reference" "DB3" (id 0) (at 172.085 99.695 0)
       (effects (font (size 1.27 1.27)) (justify left))
     )

Commit message: Changed some values on the schematic. Doesn't affect PCB
Parts:
- renumbered CB3 to CB5, CBy3 to CBy5, DB3 to DB5, LB3 to LB5, UB3v3 to UB5v0
Changed lines of the file:
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@@
     (effects (font (size 1.27 1.27)) (justify left))
   )
-  (symbol (lib_id "power:GND") (at 168.275 106.68 0)
+  (symbol (lib_id "power:GND") (at 168.275 106.68 0) (unit 1)
     (in_bom yes) (on_board yes) (fields_autoplaced)
-    (property "Reference" "#PWR0145" (id 0) (at 168.275 113.03 0)
+    (property "Reference" "#PWR0124" (id 0) (at 168.275 113.03 0)
       (effects (font (size 1.27 1.27)) hide)
     )
@@
     (pin "1")
   )
-  (symbol (lib_id "Device:C_Polarized") (at 126.365 93.98 0)
+  (symbol (lib_id "Device:C_Polarized") (at 126.365 93.98 0) (unit 1)
     (in_bom yes) (on_board yes)
-    (property "Reference" "CBy3" (id 0) (at 119.38 96.52 90)
+    (property "Reference" "CBy5" (id 0) (at 119.38 96.52 90)
       (effects (font (size 1.27 1.27)) (justify left))
     )
@@
     (pin "2")
   )
-  (symbol (lib_id "Device:C_Polarized") (at 189.865 101.6 0)
+  (symbol (lib_id "Device:C_Polarized") (at 189.865 101.6 0) (unit 1)
     (in_bom yes) (on_board yes) (fields_autoplaced)
-    (property "Reference" "CB3" (id 0) (at 193.04 99.4409 0)
+    (property "Reference" "CB5" (id 0) (at 193.04 99.4409 0)
       (effects (font (size 1.27 1.27)) (justify left))
     )
@@
     (pin "2")
   )
-  (symbol (lib_id "Device:L") (at 179.07 95.25 90)
+  (symbol (lib_id "Device:L") (at 179.07 95.25 90) (unit 1)
     (in_bom yes) (on_board yes)
-    (property "Reference" "LB3" (id 0) (at 179.705 97.79 90))
+    (property "Reference" "LB5" (id 0) (at 179.705 97.79 90))
     (property "Value" "100u" (id 1) (at 179.705 100.33 90))
     (property "Footprint" "Inductor_THT:L_Toroid_Vertical_L25.4mm_W14.7mm_P12.20mm_Vishay_TJ5_BigPads" (id 2) (at 179.07 95.25 0)
@@
     (pin "2")
   )
-  (symbol (lib_id "Regulator_Switching:LM2576S-5") (at 146.05 92.71 0)
+  (symbol (lib_id "Regulator_Switching:LM2576S-5") (at 146.05 92.71 0) (unit 1)
     (in_bom yes) (on_board yes) (fields_autoplaced)
-    (property "Reference" "UB3v3" (id 0) (at 146.05 82.55 0))
+    (property "Reference" "UB5v0" (id 0) (at 146.05 82.55 0))
     (property "Value" "LM2576S-5" (id 1) (at 146.05 85.09 0))
     (property "Footprint" "Package_TO_SOT_SMD:TO-263-5_TabPin3" (id 2) (at 146.05 99.06 0)
@@
     (pin "5")
   )
-  (symbol (lib_id "power:GND") (at 189.865 106.68 0)
+  (symbol (lib_id "power:GND") (at 189.865 106.68 0) (unit 1)
     (in_bom yes) (on_board yes) (fields_autoplaced)
-    (property "Reference" "#PWR0146" (id 0) (at 189.865 113.03 0)
+    (property "Reference" "#PWR0125" (id 0) (at 189.865 113.03 0)
       (effects (font (size 1.27 1.27)) hide)
     )
@@
     (pin "1")
   )
-  (symbol (lib_id "Diode:1N5822") (at 168.275 101.6 270)
+  (symbol (lib_id "Diode:1N5822") (at 168.275 101.6 270) (unit 1)
     (in_bom yes) (on_board yes)
-    (property "Reference" "DB3" (id 0) (at 172.085 99.695 0)
+    (property "Reference" "DB5" (id 0) (at 172.085 99.695 0)
       (effects (font (size 1.27 1.27)) (justify left))
     )
@@
     (pin "2")
   )
-  (symbol (lib_id "power:GND") (at 126.365 100.33 0)
+  (symbol (lib_id "power:GND") (at 126.365 100.33 0) (unit 1)
     (in_bom yes) (on_board yes) (fields_autoplaced)
-    (property "Reference" "#PWR0148" (id 0) (at 126.365 106.68 0)
+    (property "Reference" "#PWR0127" (id 0) (at 126.365 106.68 0)
       (effects (font (size 1.27 1.27)) hide)
     )
@@
     (pin "1")
   )
-  (symbol (lib_id "power:GND") (at 146.05 106.68 0)
+  (symbol (lib_id "power:GND") (at 146.05 106.68 0) (unit 1)
     (in_bom yes) (on_board yes) (fields_autoplaced)
-    (property "Reference" "#PWR0144" (id 0) (at 146.05 113.03 0)
+    (property "Reference" "#PWR0123" (id 0) (at 146.05 113.03 0)
       (effects (font (size 1.27 1.27)) hide)
     )
@@
     (pin "1")
   )
-  (symbol (lib_id "power:GND") (at 131.445 95.25 0)
+  (symbol (lib_id "power:GND") (at 131.445 95.25 0) (unit 1)
     (in_bom yes) (on_board yes) (fields_autoplaced)
-    (property "Reference" "#PWR0147" (id 0) (at 131.445 101.6 0)
+    (property "Reference" "#PWR0126" (id 0) (at 131.445 101.6 0)
       (effects (font (size 1.27 1.27)) hide)
     )
