File: Circuit Design/Final Schematic/Buck3v3.kicad_sch (KiCad schematic)
At the start: 0 parts

Commit message: Power Module on schematic almost ready
Parts:
- added CB3: 1u, Capacitor_SMD:CP_Elec_6.3x5.8, symbol Device:C_Polarized
- added CBy3: 100u, Capacitor_SMD:CP_Elec_6.3x5.8, symbol Device:C_Polarized
- added DB3: 1N5822, Diode_THT:D_DO-201AD_P15.24mm_Horizontal, symbol Diode:1N5822
- added LB3: 20u, Inductor_THT:L_Toroid_Vertical_L25.4mm_W14.7mm_P12.20mm_Vishay_TJ5_BigPads, symbol Device:L
- added UB5v0: LM2576S-5, Package_TO_SOT_SMD:TO-263-5_TabPin3, symbol Regulator_Switching:LM2576S-5
Connections:
- new net: DB3.1 (K), LB3.1, UB5v0.2 (OUT)
- new net GND: CB3.2, CBy3.2, DB3.2 (A), UB5v0.3 (GND), UB5v0.5 (~{ON}/OFF)
- new net Vo: CB3.1, LB3.2, UB5v0.4 (FB)
- new net v_in: CBy3.1, UB5v0.1 (VIN)
Changed lines of the file:
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@@
 (kicad_sch (version 20211123) (generator eeschema)
   (paper "A4")
+  (junction (at 168.275 95.25) (diameter 0) (color 0 0 0 0)
+  )
+  (junction (at 189.865 95.25) (diameter 0) (color 0 0 0 0)
+  )
+  (junction (at 123.19 90.17) (diameter 0) (color 0 0 0 0)
+  )
+  (wire (pts (xy 123.19 90.17) (xy 133.35 90.17))
+    (stroke (width 0) (type default) (color 0 0 0 0))
+  )
+  (wire (pts (xy 189.865 95.25) (xy 189.865 90.17))
+    (stroke (width 0) (type default) (color 0 0 0 0))
+  )
+  (wire (pts (xy 168.275 97.79) (xy 168.275 95.25))
+    (stroke (width 0) (type default) (color 0 0 0 0))
+  )
+  (wire (pts (xy 111.125 90.17) (xy 123.19 90.17))
+    (stroke (width 0) (type default) (color 0 0 0 0))
+  )
+  (wire (pts (xy 189.865 90.17) (xy 158.75 90.17))
+    (stroke (width 0) (type default) (color 0 0 0 0))
+  )
+  (wire (pts (xy 182.88 95.25) (xy 189.865 95.25))
+    (stroke (width 0) (type default) (color 0 0 0 0))
+  )
+  (wire (pts (xy 168.275 105.41) (xy 168.275 106.68))
+    (stroke (width 0) (type default) (color 0 0 0 0))
+  )
+  (wire (pts (xy 131.445 95.25) (xy 133.35 95.25))
+    (stroke (width 0) (type default) (color 0 0 0 0))
+  )
+  (wire (pts (xy 189.865 95.25) (xy 189.865 97.79))
+    (stroke (width 0) (type default) (color 0 0 0 0))
+  )
+  (wire (pts (xy 123.19 97.79) (xy 123.19 99.695))
+    (stroke (width 0) (type default) (color 0 0 0 0))
+  )
+  (wire (pts (xy 168.275 95.25) (xy 175.26 95.25))
+    (stroke (width 0) (type default) (color 0 0 0 0))
+  )
+  (wire (pts (xy 146.05 100.33) (xy 146.05 106.68))
+    (stroke (width 0) (type default) (color 0 0 0 0))
+  )
+  (wire (pts (xy 158.75 95.25) (xy 168.275 95.25))
+    (stroke (width 0) (type default) (color 0 0 0 0))
+  )
+  (wire (pts (xy 189.865 95.25) (xy 200.66 95.25))
+    (stroke (width 0) (type default) (color 0 0 0 0))
+  )
+  (wire (pts (xy 189.865 105.41) (xy 189.865 106.68))
+    (stroke (width 0) (type default) (color 0 0 0 0))
+  )
+  (hierarchical_label "v_in" (shape input) (at 111.125 90.17 180)
+    (effects (font (size 1.27 1.27)) (justify right))
+  )
+  (hierarchical_label "Vo" (shape output) (at 200.66 95.25 0)
+    (effects (font (size 1.27 1.27)) (justify left))
+  )
+  (symbol (lib_id "power:GND") (at 168.275 106.68 0) (unit 1)
+    (in_bom yes) (on_board yes) (fields_autoplaced)
+    (property "Reference" "#PWR?" (id 0) (at 168.275 113.03 0)
+      (effects (font (size 1.27 1.27)) hide)
+    )
+    (property "Value" "GND" (id 1) (at 168.275 111.76 0))
+    (property "Footprint" "" (id 2) (at 168.275 106.68 0)
+      (effects (font (size 1.27 1.27)) hide)
+    )
+    (property "Datasheet" "" (id 3) (at 168.275 106.68 0)
+      (effects (font (size 1.27 1.27)) hide)
+    )
+    (pin "1")
+  )
+  (symbol (lib_id "Device:C_Polarized") (at 123.19 93.98 0) (unit 1)
+    (in_bom yes) (on_board yes)
+    (property "Reference" "CBy3" (id 0) (at 116.205 96.52 90)
+      (effects (font (size 1.27 1.27)) (justify left))
+    )
+    (property "Value" "100u" (id 1) (at 118.745 96.52 90)
+      (effects (font (size 1.27 1.27)) (justify left))
+    )
+    (property "Footprint" "Capacitor_SMD:CP_Elec_6.3x5.8" (id 2) (at 124.1552 97.79 0)
+      (effects (font (size 1.27 1.27)) hide)
+    )
+    (property "Datasheet" "~" (id 3) (at 123.19 93.98 0)
+      (effects (font (size 1.27 1.27)) hide)
+    )
+    (pin "1")
+    (pin "2")
+  )
+  (symbol (lib_id "Device:C_Polarized") (at 189.865 101.6 0) (unit 1)
+    (in_bom yes) (on_board yes) (fields_autoplaced)
+    (property "Reference" "CB3" (id 0) (at 193.04 99.4409 0)
+      (effects (font (size 1.27 1.27)) (justify left))
+    )
+    (property "Value" "1u" (id 1) (at 193.04 101.9809 0)
+      (effects (font (size 1.27 1.27)) (justify left))
+    )
+    (property "Footprint" "Capacitor_SMD:CP_Elec_6.3x5.8" (id 2) (at 190.8302 105.41 0)
+      (effects (font (size 1.27 1.27)) hide)
+    )
+    (property "Datasheet" "~" (id 3) (at 189.865 101.6 0)
+      (effects (font (size 1.27 1.27)) hide)
+    )
+    (pin "1")
+    (pin "2")
+  )
+  (symbol (lib_id "Device:L") (at 179.07 95.25 90) (unit 1)
+    (in_bom yes) (on_board yes)
+    (property "Reference" "LB3" (id 0) (at 179.705 97.79 90))
+    (property "Value" "20u" (id 1) (at 179.705 100.33 90))
+    (property "Footprint" "Inductor_THT:L_Toroid_Vertical_L25.4mm_W14.7mm_P12.20mm_Vishay_TJ5_BigPads" (id 2) (at 179.07 95.25 0)
+      (effects (font (size 1.27 1.27)) hide)
+    )
+    (property "Datasheet" "~" (id 3) (at 179.07 95.25 0)
+      (effects (font (size 1.27 1.27)) hide)
+    )
+    (pin "1")
+    (pin "2")
+  )
+  (symbol (lib_id "Regulator_Switching:LM2576S-5") (at 146.05 92.71 0) (unit 1)
+    (in_bom yes) (on_board yes) (fields_autoplaced)
+    (property "Reference" "UB5v0" (id 0) (at 146.05 82.55 0))
+    (property "Value" "LM2576S-5" (id 1) (at 146.05 85.09 0))
+    (property "Footprint" "Package_TO_SOT_SMD:TO-263-5_TabPin3" (id 2) (at 146.05 99.06 0)
+      (effects (font (size 1.27 1.27) italic) (justify left) hide)
+    )
+    (property "Datasheet" "http://www.ti.com/lit/ds/symlink/lm2576.pdf" (id 3) (at 146.05 92.71 0)
+      (effects (font (size 1.27 1.27)) hide)
+    )
+    (pin "1")
+    (pin "2")
+    (pin "3")
+    (pin "4")
+    (pin "5")
+  )
+  (symbol (lib_id "power:GND") (at 189.865 106.68 0) (unit 1)
+    (in_bom yes) (on_board yes) (fields_autoplaced)
+    (property "Reference" "#PWR?" (id 0) (at 189.865 113.03 0)
+      (effects (font (size 1.27 1.27)) hide)
+    )
+    (property "Value" "GND" (id 1) (at 189.865 111.76 0))
+    (property "Footprint" "" (id 2) (at 189.865 106.68 0)
+      (effects (font (size 1.27 1.27)) hide)
+    )
+    (property "Datasheet" "" (id 3) (at 189.865 106.68 0)
+      (effects (font (size 1.27 1.27)) hide)
+    )
+    (pin "1")
+  )
+  (symbol (lib_id "Diode:1N5822") (at 168.275 101.6 270) (unit 1)
+    (in_bom yes) (on_board yes)
+    (property "Reference" "DB3" (id 0) (at 172.085 99.695 0)
+      (effects (font (size 1.27 1.27)) (justify left))
+    )
+    (property "Value" "1N5822" (id 1) (at 165.1 97.79 0)
+      (effects (font (size 1.27 1.27)) (justify left))
+    )
+    (property "Footprint" "Diode_THT:D_DO-201AD_P15.24mm_Horizontal" (id 2) (at 163.83 101.6 0)
+      (effects (font (size 1.27 1.27)) hide)
+    )
+    (property "Datasheet" "http://www.vishay.com/docs/88526/1n5820.pdf" (id 3) (at 168.275 101.6 0)
+      (effects (font (size 1.27 1.27)) hide)
+    )
+    (pin "1")
+    (pin "2")
+  )
+  (symbol (lib_id "power:GND") (at 123.19 99.695 0) (unit 1)
+    (in_bom yes) (on_board yes) (fields_autoplaced)
+    (property "Reference" "#PWR?" (id 0) (at 123.19 106.045 0)
+      (effects (font (size 1.27 1.27)) hide)
+    )
+    (property "Value" "GND" (id 1) (at 123.19 104.14 0))
+    (property "Footprint" "" (id 2) (at 123.19 99.695 0)
+      (effects (font (size 1.27 1.27)) hide)
+    )
+    (property "Datasheet" "" (id 3) (at 123.19 99.695 0)
+      (effects (font (size 1.27 1.27)) hide)
+    )
+    (pin "1")
+  )
+  (symbol (lib_id "power:GND") (at 146.05 106.68 0) (unit 1)
+    (in_bom yes) (on_board yes) (fields_autoplaced)
+    (property "Reference" "#PWR?" (id 0) (at 146.05 113.03 0)
+      (effects (font (size 1.27 1.27)) hide)
+    )
+    (property "Value" "GND" (id 1) (at 146.05 111.125 0))
+    (property "Footprint" "" (id 2) (at 146.05 106.68 0)
+      (effects (font (size 1.27 1.27)) hide)
+    )
+    (property "Datasheet" "" (id 3) (at 146.05 106.68 0)
+      (effects (font (size 1.27 1.27)) hide)
+    )
+    (pin "1")
+  )
+  (symbol (lib_id "power:GND") (at 131.445 95.25 0) (unit 1)
+    (in_bom yes) (on_board yes) (fields_autoplaced)
+    (property "Reference" "#PWR?" (id 0) (at 131.445 101.6 0)
+      (effects (font (size 1.27 1.27)) hide)
+    )
+    (property "Value" "GND" (id 1) (at 131.445 100.33 0))
+    (property "Footprint" "" (id 2) (at 131.445 95.25 0)
+      (effects (font (size 1.27 1.27)) hide)
+    )
+    (property "Datasheet" "" (id 3) (at 131.445 95.25 0)
+      (effects (font (size 1.27 1.27)) hide)
+    )
+    (pin "1")
+  )
 )

Commit message: Footprints
Parts:
- CB5: renamed from CB3; value 1u -> 22u
- CBy5: renamed from CBy3; value 100u -> 47u; footprint Capacitor_SMD:CP_Elec_6.3x5.8 -> Capacitor_Tantalum_SMD:CP_EIA-7343-43_Kemet-X_Pad2.25x2.55mm_HandSolder
- LB5: renamed from LB3; value 20u -> 100u
- renumbered DB3 to DB5
Other:
- moved on the sheet: CBy5
Changed lines of the file:
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@@
 (kicad_sch (version 20211123) (generator eeschema)
   (paper "A4")
+  (junction (at 126.365 90.17) (diameter 0) (color 0 0 0 0)
+  )
   (junction (at 168.275 95.25) (diameter 0) (color 0 0 0 0)
   )
   (junction (at 189.865 95.25) (diameter 0) (color 0 0 0 0)
-  )
-  (junction (at 123.19 90.17) (diameter 0) (color 0 0 0 0)
-  )
-  (wire (pts (xy 123.19 90.17) (xy 133.35 90.17))
-    (stroke (width 0) (type default) (color 0 0 0 0))
   )
   (wire (pts (xy 189.865 95.25) (xy 189.865 90.17))
@@
   )
   (wire (pts (xy 168.275 97.79) (xy 168.275 95.25))
-    (stroke (width 0) (type default) (color 0 0 0 0))
-  )
-  (wire (pts (xy 111.125 90.17) (xy 123.19 90.17))
     (stroke (width 0) (type default) (color 0 0 0 0))
   )
@@
     (stroke (width 0) (type default) (color 0 0 0 0))
   )
-  (wire (pts (xy 123.19 97.79) (xy 123.19 99.695))
+  (wire (pts (xy 126.365 90.17) (xy 133.35 90.17))
+    (stroke (width 0) (type default) (color 0 0 0 0))
+  )
+  (wire (pts (xy 126.365 97.79) (xy 126.365 100.33))
     (stroke (width 0) (type default) (color 0 0 0 0))
   )
   (wire (pts (xy 168.275 95.25) (xy 175.26 95.25))
+    (stroke (width 0) (type default) (color 0 0 0 0))
+  )
+  (wire (pts (xy 111.125 90.17) (xy 126.365 90.17))
     (stroke (width 0) (type default) (color 0 0 0 0))
   )
@@
     (pin "1")
   )
-  (symbol (lib_id "Device:C_Polarized") (at 123.19 93.98 0) (unit 1)
+  (symbol (lib_id "Device:C_Polarized") (at 126.365 93.98 0) (unit 1)
     (in_bom yes) (on_board yes)
-    (property "Reference" "CBy3" (id 0) (at 116.205 96.52 90)
+    (property "Reference" "CBy5" (id 0) (at 119.38 96.52 90)
       (effects (font (size 1.27 1.27)) (justify left))
     )
-    (property "Value" "100u" (id 1) (at 118.745 96.52 90)
+    (property "Value" "47u" (id 1) (at 121.92 96.52 90)
       (effects (font (size 1.27 1.27)) (justify left))
     )
-    (property "Footprint" "Capacitor_SMD:CP_Elec_6.3x5.8" (id 2) (at 124.1552 97.79 0)
+    (property "Footprint" "Capacitor_Tantalum_SMD:CP_EIA-7343-43_Kemet-X_Pad2.25x2.55mm_HandSolder" (id 2) (at 127.3302 97.79 0)
       (effects (font (size 1.27 1.27)) hide)
     )
-    (property "Datasheet" "~" (id 3) (at 123.19 93.98 0)
+    (property "Datasheet" "~" (id 3) (at 126.365 93.98 0)
       (effects (font (size 1.27 1.27)) hide)
     )
@@
   (symbol (lib_id "Device:C_Polarized") (at 189.865 101.6 0) (unit 1)
     (in_bom yes) (on_board yes) (fields_autoplaced)
-    (property "Reference" "CB3" (id 0) (at 193.04 99.4409 0)
+    (property "Reference" "CB5" (id 0) (at 193.04 99.4409 0)
       (effects (font (size 1.27 1.27)) (justify left))
     )
-    (property "Value" "1u" (id 1) (at 193.04 101.9809 0)
+    (property "Value" "22u" (id 1) (at 193.04 101.9809 0)
       (effects (font (size 1.27 1.27)) (justify left))
     )
@@
   (symbol (lib_id "Device:L") (at 179.07 95.25 90) (unit 1)
     (in_bom yes) (on_board yes)
-    (property "Reference" "LB3" (id 0) (at 179.705 97.79 90))
-    (property "Value" "20u" (id 1) (at 179.705 100.33 90))
+    (property "Reference" "LB5" (id 0) (at 179.705 97.79 90))
+    (property "Value" "100u" (id 1) (at 179.705 100.33 90))
     (property "Footprint" "Inductor_THT:L_Toroid_Vertical_L25.4mm_W14.7mm_P12.20mm_Vishay_TJ5_BigPads" (id 2) (at 179.07 95.25 0)
       (effects (font (size 1.27 1.27)) hide)
@@
   (symbol (lib_id "Diode:1N5822") (at 168.275 101.6 270) (unit 1)
     (in_bom yes) (on_board yes)
-    (property "Reference" "DB3" (id 0) (at 172.085 99.695 0)
+    (property "Reference" "DB5" (id 0) (at 172.085 99.695 0)
       (effects (font (size 1.27 1.27)) (justify left))
     )
@@
     (pin "2")
   )
-  (symbol (lib_id "power:GND") (at 123.19 99.695 0) (unit 1)
+  (symbol (lib_id "power:GND") (at 126.365 100.33 0) (unit 1)
     (in_bom yes) (on_board yes) (fields_autoplaced)
-    (property "Reference" "#PWR?" (id 0) (at 123.19 106.045 0)
+    (property "Reference" "#PWR?" (id 0) (at 126.365 106.68 0)
       (effects (font (size 1.27 1.27)) hide)
     )
-    (property "Value" "GND" (id 1) (at 123.19 104.14 0))
-    (property "Footprint" "" (id 2) (at 123.19 99.695 0)
+    (property "Value" "GND" (id 1) (at 126.365 104.775 0))
+    (property "Footprint" "" (id 2) (at 126.365 100.33 0)
       (effects (font (size 1.27 1.27)) hide)
     )
-    (property "Datasheet" "" (id 3) (at 123.19 99.695 0)
+    (property "Datasheet" "" (id 3) (at 126.365 100.33 0)
       (effects (font (size 1.27 1.27)) hide)
     )

Commit message: Footprints
Parts:
- renumbered CB5 to CB3, CBy5 to CBy3, DB5 to DB3, LB5 to LB3
Changed lines of the file:
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@@
     (effects (font (size 1.27 1.27)) (justify left))
   )
-  (symbol (lib_id "power:GND") (at 168.275 106.68 0) (unit 1)
+  (symbol (lib_id "power:GND") (at 168.275 106.68 0)
     (in_bom yes) (on_board yes) (fields_autoplaced)
-    (property "Reference" "#PWR?" (id 0) (at 168.275 113.03 0)
+    (property "Reference" "#PWR0145" (id 0) (at 168.275 113.03 0)
       (effects (font (size 1.27 1.27)) hide)
     )
@@
     (pin "1")
   )
-  (symbol (lib_id "Device:C_Polarized") (at 126.365 93.98 0) (unit 1)
+  (symbol (lib_id "Device:C_Polarized") (at 126.365 93.98 0)
     (in_bom yes) (on_board yes)
-    (property "Reference" "CBy5" (id 0) (at 119.38 96.52 90)
+    (property "Reference" "CBy3" (id 0) (at 119.38 96.52 90)
       (effects (font (size 1.27 1.27)) (justify left))
     )
@@
     (pin "2")
   )
-  (symbol (lib_id "Device:C_Polarized") (at 189.865 101.6 0) (unit 1)
+  (symbol (lib_id "Device:C_Polarized") (at 189.865 101.6 0)
     (in_bom yes) (on_board yes) (fields_autoplaced)
-    (property "Reference" "CB5" (id 0) (at 193.04 99.4409 0)
+    (property "Reference" "CB3" (id 0) (at 193.04 99.4409 0)
       (effects (font (size 1.27 1.27)) (justify left))
     )
@@
     (pin "2")
   )
-  (symbol (lib_id "Device:L") (at 179.07 95.25 90) (unit 1)
+  (symbol (lib_id "Device:L") (at 179.07 95.25 90)
     (in_bom yes) (on_board yes)
-    (property "Reference" "LB5" (id 0) (at 179.705 97.79 90))
+    (property "Reference" "LB3" (id 0) (at 179.705 97.79 90))
     (property "Value" "100u" (id 1) (at 179.705 100.33 90))
     (property "Footprint" "Inductor_THT:L_Toroid_Vertical_L25.4mm_W14.7mm_P12.20mm_Vishay_TJ5_BigPads" (id 2) (at 179.07 95.25 0)
@@
     (pin "2")
   )
-  (symbol (lib_id "Regulator_Switching:LM2576S-5") (at 146.05 92.71 0) (unit 1)
+  (symbol (lib_id "Regulator_Switching:LM2576S-5") (at 146.05 92.71 0)
     (in_bom yes) (on_board yes) (fields_autoplaced)
     (property "Reference" "UB5v0" (id 0) (at 146.05 82.55 0))
@@
     (pin "5")
   )
-  (symbol (lib_id "power:GND") (at 189.865 106.68 0) (unit 1)
+  (symbol (lib_id "power:GND") (at 189.865 106.68 0)
     (in_bom yes) (on_board yes) (fields_autoplaced)
-    (property "Reference" "#PWR?" (id 0) (at 189.865 113.03 0)
+    (property "Reference" "#PWR0146" (id 0) (at 189.865 113.03 0)
       (effects (font (size 1.27 1.27)) hide)
     )
@@
     (pin "1")
   )
-  (symbol (lib_id "Diode:1N5822") (at 168.275 101.6 270) (unit 1)
+  (symbol (lib_id "Diode:1N5822") (at 168.275 101.6 270)
     (in_bom yes) (on_board yes)
-    (property "Reference" "DB5" (id 0) (at 172.085 99.695 0)
+    (property "Reference" "DB3" (id 0) (at 172.085 99.695 0)
       (effects (font (size 1.27 1.27)) (justify left))
     )
@@
     (pin "2")
   )
-  (symbol (lib_id "power:GND") (at 126.365 100.33 0) (unit 1)
+  (symbol (lib_id "power:GND") (at 126.365 100.33 0)
     (in_bom yes) (on_board yes) (fields_autoplaced)
-    (property "Reference" "#PWR?" (id 0) (at 126.365 106.68 0)
+    (property "Reference" "#PWR0148" (id 0) (at 126.365 106.68 0)
       (effects (font (size 1.27 1.27)) hide)
     )
@@
     (pin "1")
   )
-  (symbol (lib_id "power:GND") (at 146.05 106.68 0) (unit 1)
+  (symbol (lib_id "power:GND") (at 146.05 106.68 0)
     (in_bom yes) (on_board yes) (fields_autoplaced)
-    (property "Reference" "#PWR?" (id 0) (at 146.05 113.03 0)
+    (property "Reference" "#PWR0144" (id 0) (at 146.05 113.03 0)
       (effects (font (size 1.27 1.27)) hide)
     )
@@
     (pin "1")
   )
-  (symbol (lib_id "power:GND") (at 131.445 95.25 0) (unit 1)
+  (symbol (lib_id "power:GND") (at 131.445 95.25 0)
     (in_bom yes) (on_board yes) (fields_autoplaced)
-    (property "Reference" "#PWR?" (id 0) (at 131.445 101.6 0)
+    (property "Reference" "#PWR0147" (id 0) (at 131.445 101.6 0)
       (effects (font (size 1.27 1.27)) hide)
     )

Commit message: Organización PCB
Parts:
- renumbered CB3 to CB5, CBy3 to CBy5, DB3 to DB5, LB3 to LB5
Changed lines of the file:
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@@
   (symbol (lib_id "power:GND") (at 168.275 106.68 0)
     (in_bom yes) (on_board yes) (fields_autoplaced)
-    (property "Reference" "#PWR0145" (id 0) (at 168.275 113.03 0)
+    (property "Reference" "#PWR0124" (id 0) (at 168.275 113.03 0)
       (effects (font (size 1.27 1.27)) hide)
     )
@@
   (symbol (lib_id "Device:C_Polarized") (at 126.365 93.98 0)
     (in_bom yes) (on_board yes)
-    (property "Reference" "CBy3" (id 0) (at 119.38 96.52 90)
+    (property "Reference" "CBy5" (id 0) (at 119.38 96.52 90)
       (effects (font (size 1.27 1.27)) (justify left))
     )
@@
   (symbol (lib_id "Device:C_Polarized") (at 189.865 101.6 0)
     (in_bom yes) (on_board yes) (fields_autoplaced)
-    (property "Reference" "CB3" (id 0) (at 193.04 99.4409 0)
+    (property "Reference" "CB5" (id 0) (at 193.04 99.4409 0)
       (effects (font (size 1.27 1.27)) (justify left))
     )
@@
   (symbol (lib_id "Device:L") (at 179.07 95.25 90)
     (in_bom yes) (on_board yes)
-    (property "Reference" "LB3" (id 0) (at 179.705 97.79 90))
+    (property "Reference" "LB5" (id 0) (at 179.705 97.79 90))
     (property "Value" "100u" (id 1) (at 179.705 100.33 90))
     (property "Footprint" "Inductor_THT:L_Toroid_Vertical_L25.4mm_W14.7mm_P12.20mm_Vishay_TJ5_BigPads" (id 2) (at 179.07 95.25 0)
@@
   (symbol (lib_id "power:GND") (at 189.865 106.68 0)
     (in_bom yes) (on_board yes) (fields_autoplaced)
-    (property "Reference" "#PWR0146" (id 0) (at 189.865 113.03 0)
+    (property "Reference" "#PWR0125" (id 0) (at 189.865 113.03 0)
       (effects (font (size 1.27 1.27)) hide)
     )
@@
   (symbol (lib_id "Diode:1N5822") (at 168.275 101.6 270)
     (in_bom yes) (on_board yes)
-    (property "Reference" "DB3" (id 0) (at 172.085 99.695 0)
+    (property "Reference" "DB5" (id 0) (at 172.085 99.695 0)
       (effects (font (size 1.27 1.27)) (justify left))
     )
@@
   (symbol (lib_id "power:GND") (at 126.365 100.33 0)
     (in_bom yes) (on_board yes) (fields_autoplaced)
-    (property "Reference" "#PWR0148" (id 0) (at 126.365 106.68 0)
+    (property "Reference" "#PWR0127" (id 0) (at 126.365 106.68 0)
       (effects (font (size 1.27 1.27)) hide)
     )
@@
   (symbol (lib_id "power:GND") (at 146.05 106.68 0)
     (in_bom yes) (on_board yes) (fields_autoplaced)
-    (property "Reference" "#PWR0144" (id 0) (at 146.05 113.03 0)
+    (property "Reference" "#PWR0123" (id 0) (at 146.05 113.03 0)
       (effects (font (size 1.27 1.27)) hide)
     )
@@
   (symbol (lib_id "power:GND") (at 131.445 95.25 0)
     (in_bom yes) (on_board yes) (fields_autoplaced)
-    (property "Reference" "#PWR0147" (id 0) (at 131.445 101.6 0)
+    (property "Reference" "#PWR0126" (id 0) (at 131.445 101.6 0)
       (effects (font (size 1.27 1.27)) hide)
     )

Commit message: PCB distribution
Parts:
- DB5: footprint Diode_THT:D_DO-201AD_P15.24mm_Horizontal -> Diode_THT:D_DO-201AE_P5.08mm_Vertical_AnodeUp
Changed lines of the file:
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@@
       (effects (font (size 1.27 1.27)) (justify left))
     )
-    (property "Footprint" "Diode_THT:D_DO-201AD_P15.24mm_Horizontal" (id 2) (at 163.83 101.6 0)
+    (property "Footprint" "Diode_THT:D_DO-201AE_P5.08mm_Vertical_AnodeUp" (id 2) (at 163.83 101.6 0)
       (effects (font (size 1.27 1.27)) hide)
     )

Commit message: Buck converters simmulations
Parts:
- CB5: value 22u -> 47u
Changed lines of the file:
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@@
       (effects (font (size 1.27 1.27)) (justify left))
     )
-    (property "Value" "22u" (id 1) (at 193.04 101.9809 0)
+    (property "Value" "47u" (id 1) (at 193.04 101.9809 0)
       (effects (font (size 1.27 1.27)) (justify left))
     )
