File: Circuit Design/Final Schematic/Report_buttons.kicad_sch (KiCad schematic)
At the start: 6 parts

Commit message: Footprints
Parts:
- removed Button_Damage?: SW_DIP_x05, symbol Switch:SW_DIP_x01
- removed Button_No_Damage?: SW_DIP_x04, symbol Switch:SW_DIP_x01
- added J_Tap_B1, J_Tap_B2, J_Tap_B3, J_Tap_B4: 62409-1, TE_62409-1, symbol Connector_Faston:62409-1
- gave numbers to parts that had none: 4
Connections:
- net +3V3: now also J_Tap_B1.1 (P1), J_Tap_B1.2 (P1), J_Tap_B2.1 (P1), J_Tap_B2.2 (P1)
- net Butt_D: now also J_Tap_B3.1 (P1), J_Tap_B3.2 (P1)
- net Butt_No_D: now also J_Tap_B4.1 (P1), J_Tap_B4.2 (P1)
Other:
- moved on the sheet: CB2, CB4, RB1, RB2

Commit message: Mounting holes
Parts:
- renumbered J_Tap_B1 to B1, J_Tap_B4 to B1_1, J_Tap_B2 to B2, J_Tap_B3 to B2_1, RB1 to RBtn1, RB2 to RBtn2
Changed lines of the file:
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@@
   (symbol (lib_id "Device:R") (at 200.66 77.47 180) (unit 1)
     (in_bom yes) (on_board yes) (fields_autoplaced)
-    (property "Reference" "RB1" (id 0) (at 203.2 76.1999 0)
+    (property "Reference" "RBtn1" (id 0) (at 203.2 76.1999 0)
       (effects (font (size 1.27 1.27)) (justify right))
     )
@@
   (symbol (lib_id "Connector_Faston:62409-1") (at 162.56 96.52 0) (unit 1)
     (in_bom yes) (on_board yes)
-    (property "Reference" "J_Tap_B2" (id 0) (at 163.83 97.79 0))
+    (property "Reference" "B2" (id 0) (at 163.83 97.79 0))
     (property "Value" "62409-1" (id 1) (at 162.56 93.98 0))
     (property "Footprint" "TE_62409-1" (id 2) (at 162.56 96.52 0)
@@
   (symbol (lib_id "Connector_Faston:62409-1") (at 160.02 69.85 0) (unit 1)
     (in_bom yes) (on_board yes)
-    (property "Reference" "J_Tap_B1" (id 0) (at 161.29 71.12 0))
+    (property "Reference" "B1" (id 0) (at 161.29 71.12 0))
     (property "Value" "62409-1" (id 1) (at 160.02 67.31 0))
     (property "Footprint" "TE_62409-1" (id 2) (at 160.02 69.85 0)
@@
   (symbol (lib_id "Connector_Faston:62409-1") (at 179.07 96.52 180) (unit 1)
     (in_bom yes) (on_board yes)
-    (property "Reference" "J_Tap_B3" (id 0) (at 177.8 95.25 0))
+    (property "Reference" "B2_1" (id 0) (at 177.8 95.25 0))
     (property "Value" "62409-1" (id 1) (at 179.07 99.06 0))
     (property "Footprint" "TE_62409-1" (id 2) (at 179.07 96.52 0)
@@
   (symbol (lib_id "Device:R") (at 200.66 104.14 180) (unit 1)
     (in_bom yes) (on_board yes) (fields_autoplaced)
-    (property "Reference" "RB2" (id 0) (at 203.2 102.8699 0)
+    (property "Reference" "RBtn2" (id 0) (at 203.2 102.8699 0)
       (effects (font (size 1.27 1.27)) (justify right))
     )
@@
   (symbol (lib_id "Connector_Faston:62409-1") (at 182.88 69.85 180) (unit 1)
     (in_bom yes) (on_board yes)
-    (property "Reference" "J_Tap_B4" (id 0) (at 181.61 68.58 0))
+    (property "Reference" "B1_1" (id 0) (at 181.61 68.58 0))
     (property "Value" "62409-1" (id 1) (at 182.88 72.39 0))
     (property "Footprint" "TE_62409-1" (id 2) (at 182.88 69.85 0)
