File: Circuit Design/Final Schematic/actuators.kicad_sch (KiCad schematic)
At the start: 2 parts

Commit message: Footprints
Parts:
- J_M1, J_M2: footprint Connector_PinHeader_2.54mm:PinHeader_1x03_P2.54mm_Vertical -> Connector_JST:JST_EH_S3B-EH_1x03_P2.50mm_Horizontal
Changed lines of the file:
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@@
   (symbol (lib_id "power:GND") (at 86.36 69.85 270) (unit 1)
     (in_bom yes) (on_board yes)
-    (property "Reference" "#PWR?" (id 0) (at 80.01 69.85 0)
+    (property "Reference" "#PWR0153" (id 0) (at 80.01 69.85 0)
       (effects (font (size 1.27 1.27)) hide)
     )
@@
   (symbol (lib_id "power:+5V") (at 86.36 57.15 90) (unit 1)
     (in_bom yes) (on_board yes) (fields_autoplaced)
-    (property "Reference" "#PWR?" (id 0) (at 90.17 57.15 0)
+    (property "Reference" "#PWR0154" (id 0) (at 90.17 57.15 0)
       (effects (font (size 1.27 1.27)) hide)
     )
@@
       (effects (font (size 1.27 1.27)) (justify left))
     )
-    (property "Footprint" "Connector_PinHeader_2.54mm:PinHeader_1x03_P2.54mm_Vertical" (id 2) (at 95.25 67.31 0)
+    (property "Footprint" "Connector_JST:JST_EH_S3B-EH_1x03_P2.50mm_Horizontal" (id 2) (at 95.25 67.31 0)
       (effects (font (size 1.27 1.27)) hide)
     )
@@
   (symbol (lib_id "power:GND") (at 86.36 59.69 270) (unit 1)
     (in_bom yes) (on_board yes)
-    (property "Reference" "#PWR?" (id 0) (at 80.01 59.69 0)
+    (property "Reference" "#PWR0155" (id 0) (at 80.01 59.69 0)
       (effects (font (size 1.27 1.27)) hide)
     )
@@
   (symbol (lib_id "power:+5V") (at 86.36 67.31 90) (unit 1)
     (in_bom yes) (on_board yes) (fields_autoplaced)
-    (property "Reference" "#PWR?" (id 0) (at 90.17 67.31 0)
+    (property "Reference" "#PWR0156" (id 0) (at 90.17 67.31 0)
       (effects (font (size 1.27 1.27)) hide)
     )
@@
       (effects (font (size 1.27 1.27)) (justify left))
     )
-    (property "Footprint" "Connector_PinHeader_2.54mm:PinHeader_1x03_P2.54mm_Vertical" (id 2) (at 95.25 57.15 0)
+    (property "Footprint" "Connector_JST:JST_EH_S3B-EH_1x03_P2.50mm_Horizontal" (id 2) (at 95.25 57.15 0)
       (effects (font (size 1.27 1.27)) hide)
     )
