File: Circuit Design/Final Schematic/perifericos.kicad_sch (KiCad schematic)
At the start: 5 parts

Commit message: Footprints
Parts:
- removed Display?: Conn_01x04_Female, Connector_PinSocket_2.54mm:PinSocket_1x04_P2.54mm_Vertical, symbol Connector:Conn_01x04_Female
- removed Display_?: Conn_01x14_Female, Connector_PinSocket_2.54mm:PinSocket_1x14_P2.54mm_Vertical, symbol Connector:Conn_01x14_Female
- added J_Display1: Conn_01x09, Connector_JST:JST_EH_S9B-EH_1x09_P2.50mm_Horizontal, symbol Connector_Generic:Conn_01x09
- J_Lector_1, J_Lector_2, J_Lector_3: renamed from J_Lector_?; footprint Connector_PinHeader_2.54mm:PinHeader_1x08_P2.54mm_Vertical -> Connector_JST:JST_EH_S8B-EH_1x08_P2.50mm_Horizontal
Connections:
- net +3V3: now also J_Display1.2 (Pin_2), J_Display1.9 (Pin_9)
- net CS_Display: now also J_Display1.7 (Pin_7)
- net D/C: now also J_Display1.5 (Pin_5)
- net GND: now also J_Display1.8 (Pin_8)
- net MISO: now also J_Display1.1 (Pin_1)
- net MOSI: now also J_Display1.4 (Pin_4)
- net Rst_D: now also J_Display1.6 (Pin_6)
- net SCK: now also J_Display1.3 (Pin_3)
- no-connect marks 12 -> 3
