File: Circuit Design/Final Schematic/PowerModule.kicad_sch (KiCad schematic)
At the start: 11 parts

Commit message: Changed some values on the schematic. Doesn't affect PCB
Parts:
- Crec1: value 100u -> 470u
- Lrec1: value 440m -> 250m
Changed lines of the file:
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@@
       (effects (font (size 1.27 1.27)) (justify left) hide)
     )
-    (property "Value" "100u" (id 1) (at 129.54 86.1059 0)
+    (property "Value" "470u" (id 1) (at 129.54 86.1059 0)
       (effects (font (size 1.27 1.27)) (justify left))
     )
@@
     (in_bom yes) (on_board yes) (fields_autoplaced)
     (property "Reference" "Lrec1" (id 0) (at 118.745 71.755 90))
-    (property "Value" "440m" (id 1) (at 118.745 74.295 90))
+    (property "Value" "250m" (id 1) (at 118.745 74.295 90))
     (property "Footprint" "Inductor_THT:L_Toroid_Vertical_L25.4mm_W14.7mm_P12.20mm_Vishay_TJ5_BigPads" (id 2) (at 118.745 77.47 0)
       (effects (font (size 1.27 1.27)) hide)

Commit message: New transformer
Parts:
- Lrec1: value 250m -> 150m
Changed lines of the file:
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@@
     (in_bom yes) (on_board yes) (fields_autoplaced)
     (property "Reference" "Lrec1" (id 0) (at 118.745 71.755 90))
-    (property "Value" "250m" (id 1) (at 118.745 74.295 90))
+    (property "Value" "150m" (id 1) (at 118.745 74.295 90))
     (property "Footprint" "Inductor_THT:L_Toroid_Vertical_L25.4mm_W14.7mm_P12.20mm_Vishay_TJ5_BigPads" (id 2) (at 118.745 77.47 0)
       (effects (font (size 1.27 1.27)) hide)
