File: Circuit Design/Final Schematic/Boost_batt.kicad_sch (KiCad schematic)
At the start: 11 parts

Commit message: Budget almost ready
Parts:
- C_b1: value C_Polarized -> 22u
Changed lines of the file:
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@@
       (effects (font (size 1.27 1.27)) (justify left))
     )
-    (property "Value" "C_Polarized" (id 1) (at 172.212 71.5009 0)
+    (property "Value" "22u" (id 1) (at 172.212 71.5009 0)
       (effects (font (size 1.27 1.27)) (justify left))
     )

Commit message: Buck converters simmulations
Parts:
- C_b1: value 22u -> 47u
Changed lines of the file:
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@@
       (effects (font (size 1.27 1.27)) (justify left))
     )
-    (property "Value" "22u" (id 1) (at 172.212 71.5009 0)
+    (property "Value" "47u" (id 1) (at 172.212 71.5009 0)
       (effects (font (size 1.27 1.27)) (justify left))
     )
